Commit message: add model urdf files

File: models/hook/Hook1/base.urdf (robot description, URDF)
Before this commit: robot base.urdf, 1 links, 0 joints
Links:
- link baseLink: geometry collision mesh filename=base.obj scale=0.7 0.7 0.7; visual mesh filename=base.obj scale=0.7 0.7 0.7

File: models/hook/Hook124/base.urdf (robot description, URDF)
Before this commit: robot base.urdf, 1 links, 0 joints
Links:
- link baseLink: geometry collision mesh filename=base.obj scale=0.7 0.7 0.7; visual mesh filename=base.obj scale=0.7 0.7 0.7

File: models/hook/Hook15/base.urdf (robot description, URDF)
Before this commit: robot base.urdf, 1 links, 0 joints
Links:
- link baseLink: geometry collision mesh filename=base.obj scale=0.4 0.4 0.4; visual mesh filename=base.obj scale=0.4 0.4 0.4

File: models/hook/Hook186/base.urdf (robot description, URDF)
Before this commit: robot base.urdf, 1 links, 0 joints
Links:
- link baseLink: geometry collision mesh filename=base.obj scale=0.8 0.8 0.8; visual mesh filename=base.obj scale=0.8 0.8 0.8

File: models/hook/Hook2/base.urdf (robot description, URDF)
Before this commit: robot base.urdf, 1 links, 0 joints
Links:
- link baseLink: geometry collision mesh filename=base.obj scale=0.6 0.6 0.6; visual mesh filename=base.obj scale=0.6 0.6 0.6

File: models/hook/Hook23/base.urdf (robot description, URDF)
Before this commit: robot base.urdf, 1 links, 0 joints
Links:
- link baseLink: geometry collision mesh filename=base.obj scale=1.5 1.5 1.5; visual mesh filename=base.obj scale=1.5 1.5 1.5

File: models/hook/Hook57/base.urdf (robot description, URDF)
Before this commit: robot base.urdf, 1 links, 0 joints
Links:
- link baseLink: geometry collision mesh filename=base.obj scale=0.9 0.9 0.9; visual mesh filename=base.obj scale=0.9 0.9 0.9

File: models/hook/Hook_long/base.urdf (robot description, URDF)
Before this commit: robot base.urdf, 1 links, 0 joints
Links:
- link baseLink: geometry collision mesh filename=base.obj scale=1 1 1; visual mesh filename=base.obj scale=1 1 1
