Commit message: fix some bugs in hanging_init_pose.py and re-collect hanging initial poses

File: models/geo_data/hanging_exp/mug_70/base.urdf (robot description, URDF)
Before this commit: robot base.urdf, 1 links, 0 joints
Links:
- link baseLink: geometry collision mesh filename=base.obj scale=0.8 0.8 0.8; visual mesh filename=base.obj scale=0.8 0.8 0.8

File: models/geo_data/hanging_exp/wrench_6/base.urdf (robot description, URDF)
Before this commit: robot base.urdf, 1 links, 0 joints
Links:
- link baseLink: geometry collision mesh filename=base.obj scale=2.5 2.5 2.5; visual mesh filename=base.obj scale=2.5 2.5 2.5
