Commit message: render multiple view affordance map and collect one trajectory for each shape

File: models/hook_all/Hook1/base.urdf (robot description, URDF)
Before this commit: robot base.urdf, 1 links, 0 joints
Links:
- link baseLink: geometry collision mesh filename=base.obj scale=1 1 1; visual mesh filename=base.obj scale=1 1 1

File: models/hook_all/Hook124/base.urdf (robot description, URDF)
Before this commit: robot base.urdf, 1 links, 0 joints
Links:
- link baseLink: geometry collision mesh filename=base.obj scale=1 1 1; visual mesh filename=base.obj scale=1 1 1

File: models/hook_all/Hook2/base.urdf (robot description, URDF)
Before this commit: robot base.urdf, 1 links, 0 joints
Links:
- link baseLink: geometry collision mesh filename=base.obj scale=1 1 1; visual mesh filename=base.obj scale=1 1 1

File: models/hook_all/Hook57/base.urdf (robot description, URDF)
Before this commit: robot base.urdf, 1 links, 0 joints
Links:
- link baseLink: geometry collision mesh filename=base.obj scale=1 1 1; visual mesh filename=base.obj scale=1 1 1
